File: board/TinyFPGA-EX.sch (KiCad schematic (older format))
At the start: 91 parts, among them J1 Conn_02x03_Odd_Even, J2 Micro_SD_Card_Det_Hirose_DM3AT, J3 USBC, J4 Conn_01x24, J5 Conn_01x24, J6 Conn_02x09_Odd_Even, J7 Conn_01x06, SW1 SW_Push, U1 LFE5UM-285, U10 PUSB3FR4Z, U11 PUSB3FR4Z, U12 DSC6001CI2A-016.0000T, U13 PL602-23, U2 S27KS0641DPBHI020, U3 DSC6001CI2A-016.0000T, U4 FAN53555, U5 MIC5504-2.5YMT-TR, U6 MIC5504-1.8YMT-TR, U7 FAN53600, U8 S25FL064L, U9 MIC5504-1.2YMT-TR

Commit message: latest tweaks
Parts:
- removed C21: 1uF, Footprints:C_0402_NoSilk, symbol Device:C_Small
- removed C25, C27: 10nf, Footprints:C_0402_NoSilk, symbol Device:C_Small
- removed C32, C48: 100nF, Footprints:C_0402_NoSilk, symbol Device:C_Small
- removed C49: 10nF, Footprints:C_0402_NoSilk, symbol Device:C_Small
- removed R1, R2: 100, Footprints:R_0402_NoSilk, symbol Device:R_Small
- removed TP14: TEST, Footprints:small-testpoint, symbol Connector:Test_Point
- removed U12: DSC6001CI2A-016.0000T, Footprints:CDFN3225-4LD-PL-1, symbol Components:DSC6001CI2A-016.0000T
- removed U13: PL602-23, symbol Connector_Generic:Conn_02x03_Counter_Clockwise
- removed U6: MIC5504-1.8YMT-TR, Footprints:Thin-DFN4, symbol Components:MIC5504-1.8YM5-TR
- added U6: Conn_02x03_Counter_Clockwise, symbol Connector_Generic:Conn_02x03_Counter_Clockwise
- C18: value 1uF -> 100nF
- J6: symbol Connector_Generic:Conn_02x09_Odd_Even -> Connector_Generic:Conn_02x11_Odd_Even
Connections:
- net labels added: PIN50, PIN51, PIN52, PIN53, PIN54, PIN55
- net labels removed: +1V8, CLK_25MHz, RAM_CK-
- wire segments 518 -> 475
Other:
- note removed: "1.8 Volt LDO Regulator"
- moved on the sheet: C24, C26
