File: board/TinyFPGA-EX.kicad_pcb (KiCad board)
At the start: 6 copper layers, 17.8 x 61 mm, 95 parts, among them J1 Conn_02x03_Odd_Even, J2 Micro_SD_Card_Det_Hirose_DM3AT, J3 USBC, J4 Conn_01x24, J5 Conn_01x24, J6 Conn_02x09_Odd_Even, J7 Conn_01x06, SW1 SW_Push, U1 LFE5UM-285, U10 PUSB3FR4Z, U11 PUSB3FR4Z, U12 DSC6001CI2A-016.0000T, U13 PL602-23, U2 S27KS0641DPBHI020, U3 DSC6001CI2A-016.0000T, U4 FAN53555, U5 MIC5504-2.5YMT-TR, U6 MIC5504-1.8YMT-TR, U7 FAN53600, U8 S25FL064L, U9 MIC5504-1.2YMT-TR

Commit message: latest tweaks
Parts:
- removed C21: 1uF, Footprints:C_0402_NoSilk
- removed C25, C27: 10nf, Footprints:C_0402_NoSilk
- removed C32, C48: 100nF, Footprints:C_0402_NoSilk
- removed C49: 10nF, Footprints:C_0402_NoSilk
- removed J7: Conn_01x06, Pin_Headers:Pin_Header_Straight_1x06_Pitch1.27mm_SMD_Pin1Left
- removed R1, R2: 100, Footprints:R_0402_NoSilk
- removed the TP12 at (131.9, 76.4)
- removed TP14: TEST, Footprints:small-testpoint
- removed U12: DSC6001CI2A-016.0000T, Footprints:DSC6001HI2A
- removed U13: PL602-23, tinyfpga_boards:SOT-23-6
- added REF**: , Footprints:R_0603_HandSoldering, B.Cu at (137.3, 53.4)
- added REF**: , Footprints:R_0603_HandSoldering, B.Cu at (138.6, 53.4)
- added REF**: , Footprints:R_0603_HandSoldering, B.Cu at (134.5, 53.4)
- added REF**: , Footprints:R_0603_HandSoldering, B.Cu at (133.2, 53.4)
- added TP12: TEST, Footprints:small-testpoint, B.Cu at (135.1, 57.1)
- added TP12: TEST, Footprints:small-testpoint, B.Cu at (137.0, 56.6)
- added TP12: TEST, Footprints:small-testpoint, B.Cu at (136.0, 52.6)
- added TP12: TEST, Footprints:small-testpoint, B.Cu at (135.8, 54.6)
- added TP12: TEST, Footprints:small-testpoint, B.Cu at (132.6, 71.0)
- added TP12: TEST, Footprints:small-testpoint, B.Cu at (130.1, 58.6)
- added TP12: TEST, Footprints:small-testpoint, B.Cu at (134.7, 71.0)
- added TP12: TEST, Footprints:small-testpoint, B.Cu at (135.1, 72.8)
- added TP12: TEST, Footprints:small-testpoint, B.Cu at (132.8, 76.8)
- C10, C11, C12, C13, C14, C15, C16, C28, C29, C3, C30, C31, C34, C35, C36, C38, C39, C4, C40, C41, C44, C45, C46, C47, C6, C7, C9: footprint Footprints:C_0402_NoSilk -> Footprints:C_0201_NoSilk
- C18: value 1uF -> 100nF; footprint Footprints:C_0402_NoSilk -> Footprints:C_0201_NoSilk
- C24, C26: footprint Footprints:C_0402_NoSilk -> Footprints:C_0201_NoSilk; moved to F.Cu
- C37: footprint Footprints:C_0402_NoSilk -> Capacitors_SMD:C_0201_NoSilk
- J6: footprint Pin_Headers:Pin_Header_Straight_2x09_Pitch2.54mm_SMD -> Pin_Headers:Pin_Header_Straight_2x11_Pitch2.54mm_SMD
- R12, R13: value 270 -> 4.7K
- R5, R7: footprint Footprints:R_0402_NoSilk -> Footprints:R_0201_NoSilk
- U6: value MIC5504-1.8YMT-TR -> Conn_02x03_Counter_Clockwise; footprint Footprints:Thin-DFN4 -> Footprints:ASG2-D-X-B
- moved U6 8.51 mm to (140.2, 81.4), turned to 315 degrees
- moved C18 7.94 mm to (138.2, 82.0), turned to 225 degrees
- moved C24 7.43 mm to (140.4, 94.9), turned to 0 degrees
- moved REF*** 4.31 mm to (131.3, 81.9)
- moved J6 2.54 mm to (137.2, 97.8)
- moved C3 2.28 mm to (138.9, 78.4), turned to 135 degrees
- moved C26 2.11 mm to (135.3, 90.1)
- moved C40 1.93 mm to (139.1, 76.8)
- moved C4 1.62 mm to (138.4, 78.8), turned to 135 degrees
- moved C30 1.47 mm to (134.3, 78.1)
- moved C6 1.41 mm to (137.1, 75.2), turned to 315 degrees
- moved R5 1.36 mm to (136.0, 74.3), turned to 0 degrees
- moved R7 1.18 mm to (135.1, 74.1), turned to 270 degrees
- moved C39 1.07 mm to (138.2, 75.8)
- moved C10 0.95 mm to (136.7, 76.8)
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Connections:
- C24 pad 1: VCCIO3 -> VCCIO0
- C26 pad 1: VCCIO3 -> VCCIO0
- C3 pad 1: VCCIO3 -> VCCIO0
- C4 pad 1: VCCIO3 -> VCCIO0
- D2 pad 2: PIN45 -> PIN48
- J3 pad G: (no net) -> GND
- J6 pad 10: PIN46 -> PIN49
- J6 pad 11: PIN45 -> PIN48
- J6 pad 12: PIN47 -> PIN50
- J6 pad 13: PIN44 -> PIN47
- J6 pad 14: PIN48 -> PIN51
- J6 pad 15: PIN43 -> PIN46
- J6 pad 16: PIN49 -> PIN52
- U1 pad A2: PIN46 -> PIN49
- U1 pad A6: PIN44 -> PIN47
- U1 pad A7: PIN45 -> PIN48
- U1 pad B2: PIN47 -> PIN50
- U1 pad B4: PIN48 -> PIN51
- U1 pad B6: PIN43 -> PIN46
- U1 pad C3: Net-(U1-PadC3) -> PIN43
- U1 pad D2: PIN49 -> PIN52
- U1 pad F1: RAM_DQ6 -> RAM_CK+
- U1 pad F2: RAM_CK- -> RAM_DQ6
- U1 pad F4: Net-(U1-PadF4) -> PIN44
- U1 pad G3: GND -> Net-(U1-PadG3)
- U1 pad G4: Net-(U1-PadG4) -> VCCIO0
- U1 pad H1: RAM_CK+ -> RAM_CS_B
- U1 pad H2: GND -> Net-(U1-PadH2)
- U1 pad H3: GND -> Net-(U1-PadH3)
- U1 pad H4: Net-(U1-PadH4) -> VCCIO0
- U1 pad J1: RAM_DQ5 -> RAM_DQ0
- U1 pad J2: GND -> RAM_RWDS
- U1 pad K1: RAM_CS_B -> RAM_DQ2
- U1 pad K2: GND -> RAM_RESET_B
- U1 pad L1: RAM_RWDS -> RAM_DQ5
- U1 pad M1: RAM_DQ0 -> RAM_DQ4
- U1 pad M2: GND -> RAM_DQ3
- U1 pad M5: VCCIO3 -> VCCIO0
- U1 pad N1: RAM_RESET_B -> PIN55
- U1 pad N2: RAM_DQ2 -> PIN54
- U1 pad N3: RAM_DQ3 -> PIN53
- U1 pad N4: RAM_DQ4 -> PIN45
- U1 pad N5: VCCIO3 -> VCCIO0
- U2 pad B1: RAM_CK- -> Net-(U2-PadB1)
- U2 pad B4: VCCIO3 -> VCCIO0
- U2 pad D1: VCCIO3 -> VCCIO0
- U2 pad E4: VCCIO3 -> VCCIO0
- U6 pad 1: VCCIO3 -> VCCIO0
- U6 pad 2: GND -> Net-(U6-Pad2)
- U6 pad 3: VCCIO0 -> GND
- U6 pad 4: VCCIO0 -> USB3_REFCLK_0
Routing:
- net GND: track 181.8 -> 162.5 mm, vias 70 -> 65
- net PIN50: track 0.00 -> 18.5 mm, vias 0 -> 2
- net PIN51: track 0.00 -> 15.8 mm, vias 0 -> 2
- net PIN53: track 0.00 -> 15.6 mm, vias 0 -> 1
- net (no net): track 0.00 -> 13.3 mm
- net PIN52: track 0.00 -> 11.5 mm, vias 0 -> 2
- net VCCIO3: track 9.90 -> 0.00 mm, vias 4 -> 0
- net PIN43: track 14.7 -> 5.34 mm
- net PIN54: track 0.00 -> 8.70 mm, vias 0 -> 1
- net PIN49: track 10.1 -> 18.7 mm
- net RAM_CK-: track 8.54 -> 0.00 mm
- net PIN44: track 15.8 -> 7.32 mm
- net PIN48: track 14.9 -> 23.3 mm
- net +1V2A: track 14.1 -> 8.46 mm
- net PROGRAMN: track 42.1 -> 47.5 mm
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- added copper zone on B.Cu, net +1V2A
- added copper zone on B.Cu, net GND
- removed copper zone on PWR.Cu, net VCCIO3
Other:
- board text added: "3v"
- board text added: "50"
- board text added: "51"
- board text added: "52"
- board text added: "53"
- board text added: "54"
- board text added: "55"

Commit message: minor updates for rev c
Parts:
- C8: footprint Footprints:C_0402_NoSilk -> Footprints:C_0201_NoSilk
- R3, R8: footprint Footprints:R_0402_NoSilk -> Footprints:R_0201_NoSilk
- moved R4 0.75 mm to (134.2, 65.8)
- moved R3 0.38 mm to (134.9, 62.7)
- moved R8 0.08 mm to (134.9, 62.2)
Connections:
- J3 pad G: GND -> (no net)
Routing:
- net TCK: track 12.7 -> 13.5 mm
- net GND: track 162.5 -> 163.3 mm
- net USB3_REFCLK_1: track 3.74 -> 4.53 mm
